File: Eagle Design/BLE Development Board v2.1.brd (EAGLE design)
At the start: 40.1 x 22.9 mm, 24 parts, among them U2 MCP1700, U3 HM-10

Commit message: improved version
Parts:
- moved PWR 0.25 mm to (7.62, 18.3)
- moved R3 0.25 mm to (5.59, 17.5)
- moved R4 0.25 mm to (13.0, 18.3)
- moved USR 0.25 mm to (10.2, 18.3)
Other:
- board size 40.1 x 22.9 mm -> 40.4 x 22.9 mm
- board text added: "5V GND 3.3V RES P20 P21 P22 U- U+ P15 P14 P17 P16"
- board text added: "BLE"
- board text added: "Bluetooth 4.0"
- board text added: "CC2540"
- board text added: "v 2.1"
- board text removed: "5V GND 3.3V RES P20 P21 P22 U- U+ P15 P15 P17 P16"
- board text removed: "BLE 4.0"
